Commit message: Add ur_manipulator_with_vg10 group

File: neo_ur_moveit_config/srdf/vg10.srdf.xacro (robot description, xacro)
@@ -16,4 +16,13 @@
     <disable_collisions link1="vg10" link2="${prefix_value}wrist_3_link" reason="Adjacent" />
     <disable_collisions link1="vg10" link2="vg10_quick_changer" reason="Adjacent" />
+    <group name="vg10">
+      <joint name="vg10_quick_changer_joint"/>
+      <joint name="vg10_mount_joint"/>
+      <joint name="vg10_grasp_center_joint"/>
+    </group>
+    <group name="ur_manipulator_with_vg10">
+      <group name="ur_manipulator"/>
+      <group name="vg10"/>
+    </group>
   </xacro:macro>
 </robot>
