Commit message: Add custom home position

File: neo_ur_moveit_config/srdf/mpo_700.srdf.xacro (robot description, xacro)
@@ -38,4 +38,12 @@
       <joint name="${prefix_value}wrist_2_joint" value="-1.6" />
       <joint name="${prefix_value}wrist_3_joint" value="-0.11" />
+    </group_state>
+    <group_state name="home" group="ur_manipulator">
+      <joint name="${prefix_value}shoulder_pan_joint" value="${pi / 2}" />
+      <joint name="${prefix_value}shoulder_lift_joint" value="${-pi / 2}" />
+      <joint name="${prefix_value}elbow_joint" value="${-pi * 3 / 4}" />
+      <joint name="${prefix_value}wrist_1_joint" value="${-pi * 3 / 4}" />
+      <joint name="${prefix_value}wrist_2_joint" value="${-pi/2}" />
+      <joint name="${prefix_value}wrist_3_joint" value="0" />
     </group_state>
     <!--DISABLE COLLISIONS: By default it is assumed that any link of the robot could potentially come into collision with any other link in the robot. This tag disables collision checking between a specified pair of links. -->

Commit message: Add 'forward' named state

File: neo_ur_moveit_config/srdf/mpo_700.srdf.xacro (robot description, xacro)
@@ -45,4 +45,12 @@
       <joint name="${prefix_value}wrist_1_joint" value="${-pi * 3 / 4}" />
       <joint name="${prefix_value}wrist_2_joint" value="${-pi/2}" />
+      <joint name="${prefix_value}wrist_3_joint" value="0" />
+    </group_state>
+    <group_state name="forward" group="ur_manipulator">
+      <joint name="${prefix_value}shoulder_pan_joint" value="-1.2202613989459437" />
+      <joint name="${prefix_value}shoulder_lift_joint" value="-1.5495208718678732" />
+      <joint name="${prefix_value}elbow_joint" value="-2.1362695693969727" />
+      <joint name="${prefix_value}wrist_1_joint" value="-2.5972725353636683" />
+      <joint name="${prefix_value}wrist_2_joint" value="-1.2178118864642542" />
       <joint name="${prefix_value}wrist_3_joint" value="0" />
     </group_state>

Commit message: Add disable_scanners option
Silence missing lidar link warnings when disable_scanners is used with
the URDF.

File: neo_ur_moveit_config/srdf/mpo_700.srdf.xacro (robot description, xacro)
@@ -7,6 +7,8 @@
     <xacro:arg name="prefix" default=""/>
     <xacro:arg name="gripper_type" default=""/>
+    <xacro:arg name="disable_scanners" default="false"/>
     <xacro:property name="prefix_value" value="$(arg prefix)"/>
     <xacro:property name="gripper" value="$(arg gripper_type)"/>
+    <xacro:property name="disable_scanners" value="$(arg disable_scanners)"/>
     <!--GROUPS: Representation of a set of joints and links. This can be useful for specifying DOF to plan for, defining arms, end effectors, etc-->
     <!--LINKS: When a link is specified, the parent joint of that link (if it exists) is automatically included-->
@@ -57,6 +59,4 @@
     <!--DISABLE COLLISIONS: By default it is assumed that any link of the robot could potentially come into collision with any other link in the robot. This tag disables collision checking between a specified pair of links. -->
     <disable_collisions link1="base_footprint" link2="cabinet_link" reason="Adjacent"/>
-    <disable_collisions link1="base_footprint" link2="lidar_1_link" reason="Adjacent"/>
-    <disable_collisions link1="base_footprint" link2="lidar_2_link" reason="Adjacent"/>
     <disable_collisions link1="base_footprint" link2="caster_back_left_link" reason="Adjacent"/>
     <disable_collisions link1="base_footprint" link2="caster_back_right_link" reason="Adjacent"/>
@@ -69,6 +69,4 @@
     <disable_collisions link1="base_footprint" link2="${prefix_value}base_link_inertia" reason="Never"/>
     <disable_collisions link1="base_footprint" link2="${prefix_value}shoulder_link" reason="Never"/>
-    <disable_collisions link1="cabinet_link" link2="lidar_1_link" reason="Adjacent"/>
-    <disable_collisions link1="cabinet_link" link2="lidar_2_link" reason="Adjacent"/>
     <disable_collisions link1="cabinet_link" link2="caster_back_left_link" reason="Never"/>
     <disable_collisions link1="cabinet_link" link2="caster_back_right_link" reason="Never"/>
@@ -81,26 +79,32 @@
     <disable_collisions link1="cabinet_link" link2="${prefix_value}base_link_inertia" reason="Adjacent"/>
     <disable_collisions link1="cabinet_link" link2="${prefix_value}shoulder_link" reason="Never"/>
-    <disable_collisions link1="lidar_1_link" link2="lidar_2_link" reason="Adjacent"/>
-    <disable_collisions link1="lidar_1_link" link2="caster_back_left_link" reason="Never"/>
-    <disable_collisions link1="lidar_1_link" link2="caster_back_right_link" reason="Never"/>
-    <disable_collisions link1="lidar_1_link" link2="caster_front_left_link" reason="Never"/>
-    <disable_collisions link1="lidar_1_link" link2="caster_front_right_link" reason="Never"/>
-    <disable_collisions link1="lidar_1_link" link2="wheel_back_left_link" reason="Never"/>
-    <disable_collisions link1="lidar_1_link" link2="wheel_back_right_link" reason="Never"/>
-    <disable_collisions link1="lidar_1_link" link2="wheel_front_left_link" reason="Never"/>
-    <disable_collisions link1="lidar_1_link" link2="wheel_front_right_link" reason="Never"/>
-    <disable_collisions link1="lidar_1_link" link2="${prefix_value}base_link_inertia" reason="Never"/>
-    <disable_collisions link1="lidar_1_link" link2="${prefix_value}shoulder_link" reason="Never"/>
-    <disable_collisions link1="lidar_2_link" link2="caster_back_left_link" reason="Never"/>
-    <disable_collisions link1="lidar_2_link" link2="caster_back_right_link" reason="Never"/>
-    <disable_collisions link1="lidar_2_link" link2="caster_front_left_link" reason="Never"/>
-    <disable_collisions link1="lidar_2_link" link2="caster_front_right_link" reason="Never"/>
-    <disable_collisions link1="lidar_2_link" link2="wheel_back_left_link" reason="Never"/>
-    <disable_collisions link1="lidar_2_link" link2="wheel_back_right_link" reason="Never"/>
-    <disable_collisions link1="lidar_2_link" link2="wheel_front_left_link" reason="Never"/>
-    <disable_collisions link1="lidar_2_link" link2="wheel_front_right_link" reason="Never"/>
-    <disable_collisions link1="lidar_2_link" link2="${prefix_value}base_link_inertia" reason="Never"/>
-    <disable_collisions link1="lidar_2_link" link2="${prefix_value}shoulder_link" reason="Never"/>
-    <disable_collisions link1="lidar_2_link" link2="${prefix_value}upper_arm_link" reason="Never"/>
+    <xacro:if value="${disable_scanners == False}">
+      <disable_collisions link1="base_footprint" link2="lidar_1_link" reason="Adjacent"/>
+      <disable_collisions link1="base_footprint" link2="lidar_2_link" reason="Adjacent"/>
+      <disable_collisions link1="cabinet_link" link2="lidar_1_link" reason="Adjacent"/>
+      <disable_collisions link1="cabinet_link" link2="lidar_2_link" reason="Adjacent"/>
+      <disable_collisions link1="lidar_1_link" link2="lidar_2_link" reason="Adjacent"/>
+      <disable_collisions link1="lidar_1_link" link2="caster_back_left_link" reason="Never"/>
+      <disable_collisions link1="lidar_1_link" link2="caster_back_right_link" reason="Never"/>
+      <disable_collisions link1="lidar_1_link" link2="caster_front_left_link" reason="Never"/>
+      <disable_collisions link1="lidar_1_link" link2="caster_front_right_link" reason="Never"/>
+      <disable_collisions link1="lidar_1_link" link2="wheel_back_left_link" reason="Never"/>
+      <disable_collisions link1="lidar_1_link" link2="wheel_back_right_link" reason="Never"/>
+      <disable_collisions link1="lidar_1_link" link2="wheel_front_left_link" reason="Never"/>
+      <disable_collisions link1="lidar_1_link" link2="wheel_front_right_link" reason="Never"/>
+      <disable_collisions link1="lidar_1_link" link2="${prefix_value}base_link_inertia" reason="Never"/>
+      <disable_collisions link1="lidar_1_link" link2="${prefix_value}shoulder_link" reason="Never"/>
+      <disable_collisions link1="lidar_2_link" link2="caster_back_left_link" reason="Never"/>
+      <disable_collisions link1="lidar_2_link" link2="caster_back_right_link" reason="Never"/>
+      <disable_collisions link1="lidar_2_link" link2="caster_front_left_link" reason="Never"/>
+      <disable_collisions link1="lidar_2_link" link2="caster_front_right_link" reason="Never"/>
+      <disable_collisions link1="lidar_2_link" link2="wheel_back_left_link" reason="Never"/>
+      <disable_collisions link1="lidar_2_link" link2="wheel_back_right_link" reason="Never"/>
+      <disable_collisions link1="lidar_2_link" link2="wheel_front_left_link" reason="Never"/>
+      <disable_collisions link1="lidar_2_link" link2="wheel_front_right_link" reason="Never"/>
+      <disable_collisions link1="lidar_2_link" link2="${prefix_value}base_link_inertia" reason="Never"/>
+      <disable_collisions link1="lidar_2_link" link2="${prefix_value}shoulder_link" reason="Never"/>
+      <disable_collisions link1="lidar_2_link" link2="${prefix_value}upper_arm_link" reason="Never"/>
+    </xacro:if>
     <disable_collisions link1="caster_back_left_link" link2="caster_back_right_link" reason="Never"/>
     <disable_collisions link1="caster_back_left_link" link2="caster_front_left_link" reason="Never"/>
